File: chilly_board.kicad_sch (KiCad schematic)
At the start: 8 parts, among them U2 ESP32-S3

Commit message: Finally finished the schematic!!!
Parts:
- removed C1: C, symbol Device:C
- removed D1: ESD, symbol Device:D_TVS_Filled
- removed L1: L, symbol Device:L
- removed U2: ESP32-S3, Package_DFN_QFN:QFN-56-1EP_7x7mm_P0.4mm_EP4x4mm, symbol MCU_Espressif:ESP32-S3
- added +3V3: +3V3, TestPoint:TestPoint_Pad_D1.0mm, symbol Connector:TestPoint
- added AE1: Antenna, RF_Antenna:Texas_SWRA117D_2.4GHz_Left, symbol Device:Antenna_Chip
- added BTN1: BTN, Button_Switch_SMD:SW_Push_1P1T_XKB_TS-1187A, symbol Switch:SW_Push
- added C10, C11, C15, C18, C19, C32, C35: 0.1uF, Capacitor_SMD:C_0402_1005Metric, symbol Device:C
- added C13, C26, C39: 1uF, Capacitor_SMD:C_0402_1005Metric, symbol Device:C
- added C14: DNP, Capacitor_SMD:C_0402_1005Metric, symbol Device:C
- added C16, C17, C2, C25, C36, C6, C7, C8: 10uF, Capacitor_SMD:C_0402_1005Metric, symbol Device:C
- added C31, DNP1: 15pF, Capacitor_SMD:C_0402_1005Metric, symbol Device:C
- added C33, C37, C38, C4: 12pF, Capacitor_SMD:C_0402_1005Metric, symbol Device:C
- added C40: 10nF, Capacitor_SMD:C_0402_1005Metric, symbol Device:C
- added D1, D2, D3: LED, LED_SMD:LED_0603_1608Metric, symbol Device:LED
- added D4: SS14, Diode_SMD:D_SMA, symbol Diode:SS14
- added Flash1: Flash, Button_Switch_SMD:SW_Push_1P1T_XKB_TS-1187A, symbol Switch:SW_Push
- added GND1: GND, TestPoint:TestPoint_Pad_D1.0mm, symbol Connector:TestPoint
- added J1: USB_C_Receptacle_USB2.0_14P, Connector_USB:USB_C_Receptacle_HCTL_HC-TYPE-C-16P-01A, symbol Connector:USB_C_Receptacle_USB2.0_14P
- added J2: Conn_01x02_Pin, Connector_PinSocket_2.54mm:PinSocket_1x02_P2.54mm_Vertical, symbol Connector:Conn_01x02_Pin
- added J3, J5: Conn_01x18_Pin, Connector_PinHeader_2.54mm:PinHeader_1x18_P2.54mm_Vertical, symbol Connector:Conn_01x18_Pin
- added L3: 2nH, Inductor_SMD:L_0402_1005Metric, symbol Device:L
- added L5: DNP, Inductor_SMD:L_0402_1005Metric, symbol Device:L
- added L6: 4.7nH, Inductor_SMD:L_0402_1005Metric, symbol Device:L
- added Q1: AO3401A, Package_TO_SOT_SMD:SOT-23, symbol Transistor_FET:AO3401A
- added R12, R19: 200K, Resistor_SMD:R_0402_1005Metric, symbol Device:R
- added R14, R17: 5.1K, Resistor_SMD:R_0402_1005Metric, symbol Device:R
- added R15: 1K, Resistor_SMD:R_0402_1005Metric, symbol Device:R
- added R16, R24, R25: 470R, Resistor_SMD:R_0402_1005Metric, symbol Device:R
- added R18, R2: 33R, Resistor_SMD:R_0402_1005Metric, symbol Device:R
- added R20: 100K, Resistor_SMD:R_0402_1005Metric, symbol Device:R
- added R21, R22, R4: 10K, Resistor_SMD:R_0402_1005Metric, symbol Device:R
- added R23, R26, R27, R28, R29, R30: 0R, Resistor_SMD:R_0402_1005Metric, symbol Device:R
- added R31: DNP, Resistor_SMD:R_0402_1005Metric, symbol Device:R
- added Reset1: Reset, Button_Switch_SMD:SW_Push_1P1T_XKB_TS-1187A, symbol Switch:SW_Push
- added U1: ESP32-S3, Package_DFN_QFN:QFN-56-1EP_7x7mm_P0.4mm_EP4x4mm, symbol MCU_Espressif:ESP32-S3
- added U2: W25Q128JVS, Package_SO:SOIC-8_5.3x5.3mm_P1.27mm, symbol Memory_Flash:W25Q128JVS
- added U3: MCP73831-2-OT, Package_TO_SOT_SMD:SOT-23-5, symbol Battery_Management:MCP73831-2-OT
- added U4: AMS1117-3.3, Package_TO_SOT_SMD:SOT-223-3_TabPin2, symbol Regulator_Linear:AMS1117-3.3
- added Y1: 32.768 kHz, Crystal:Crystal_SMD_3215-2Pin_3.2x1.5mm, symbol Device:Crystal
- added Y2: 40MHz(10ppm), Crystal:Crystal_SMD_2520-4Pin_2.5x2.0mm, symbol Device:Crystal_GND24
- C20: value 1uF -> 10uF; footprint (none) -> Capacitor_SMD:C_0402_1005Metric; LCSC (none) -> C15525; MNF PART NUMBER (none) -> C15525
- C22: value 10uF -> 0.1uF; footprint (none) -> Capacitor_SMD:C_0402_1005Metric; LCSC (none) -> C1525; MNF PART NUMBER (none) -> C1525
- C3: value 100pF -> 10uF; footprint (none) -> Capacitor_SMD:C_0402_1005Metric; LCSC (none) -> C15525; MNF PART NUMBER (none) -> C15525
- R1: value R -> 2K; footprint (none) -> Resistor_SMD:R_0402_1005Metric; LCSC (none) -> C4109; MNF PART NUMBER (none) -> C4109
Connections:
- net GND: now also R1.1, AE1.2 (PCB_Trace), BTN1.1, C10.2, C11.2, C13.2, C14.2, C15.2, C16.2, C17.2, C18.2, C19.2, C2.2, C25.2, C26.2, C31.2, C32.2, C33.1, C35.2, C36.2, C37.2, C38.2, C39.2, C4.2, C40.2, C6.2, C7.2, C8.2, DNP1.2, Flash1.1, GND1.1, J1.A1 (GND), J1.A12 (GND), J1.B1 (GND), J1.B12 (GND), J1.S1 (SHIELD), J2.1 (Pin_1), J3.17 (Pin_17), J3.18 (Pin_18), R14.1, R16.2, R17.1, R19.2, R20.1, R25.2, Reset1.1, U1.57 (GND), U2.4 (GND), U3.2 (V_{SS}), U4.1 (GND), Y2.2, Y2.4
- net at R1.2: now also U3.5 (PROG)
- net VDD33 renamed +3V3
- net +3V3: now also +3V3.1, C10.1, C11.1, C17.1, C18.1, C25.1, C26.1, C35.1, C39.1, C40.1, D2.2 (A), J3.15 (Pin_15), L3.1, R21.1, R22.2, R31.2, R4.1, U1.20 (VDD3P3_RTC), U1.46 (VDD3P3_CPU), U1.55 (VDDA), U1.56 (VDDA), U4.2 (VO); no longer C22.1
- new net: R24.1, U1.49 (U0TXD)
- new net: J1.A5 (CC1), R14.2
- new net: J1.B5 (CC2), R17.2
- new net: D2.1 (K), R16.1
- new net: R28.1, U1.33 (SPICLK)
- new net: C14.1, L5.1
- new net: AE1.1 (FEED), C31.1, L5.2, L6.2
- new net: R29.1, U1.31 (SPIWP)
- new net: C4.1, R23.1, Y2.1
- new net: DNP1.1, L6.1, U1.1 (LNA_IN)
- new net: R27.1, U1.34 (SPIQ)
- new net: C19.1, L3.2, U1.2 (VDD3P3), U1.3 (VDD3P3)
- new net: R30.1, U1.30 (SPIHD)
- new net: R26.1, U1.35 (SPID)
- new net: C33.2, U1.53 (XTAL_N), Y2.3
- new net: R23.2, U1.54 (XTAL_P)
- new net: R15.1, U3.1 (STAT)
- new net: D1.1 (K), R15.2
- new net: D3.1 (K), R25.1
- new net 5V: C16.1, C22.1, C36.1, C6.1, D1.2 (A), D4.2 (A), J1.A4 (VBUS), J1.A9 (VBUS), J1.B4 (VBUS), J1.B9 (VBUS), J3.16 (Pin_16), Q1.1 (G), R20.2, U3.4 (V_{DD})
- new net EN: C15.1, R22.1, Reset1.2, U1.4 (CHIP_PU)
- new net IO0: Flash1.2, J5.1 (Pin_1), R21.2, U1.5 (GPIO0)
- new net IO1: D3.2 (A), U1.6 (GPIO1)
- new net IO10: J3.3 (Pin_3), U1.15 (GPIO10)
- new net IO11: J3.4 (Pin_4), U1.16 (GPIO11)
- new net IO12: J3.9 (Pin_9), U1.17 (GPIO12)
- new net IO13: J3.10 (Pin_10), U1.18 (GPIO13)
- new net IO14: BTN1.2, J3.11 (Pin_11), R4.2, U1.19 (GPIO14)
- new net IO17/SCL: J3.12 (Pin_12), U1.23 (GPIO17)
- new net IO18/SDA: J3.13 (Pin_13), U1.24 (GPIO18)
- new net IO2: J5.2 (Pin_2), U1.7 (GPIO2)
- new net IO21: J3.14 (Pin_14), U1.27 (GPIO21)
- new net IO3: J3.5 (Pin_5), U1.8 (GPIO3)
- new net IO33: J5.17 (Pin_17), U1.38 (GPIO33)
- new net IO34: J5.16 (Pin_16), U1.39 (GPIO34)
- new net IO35: J5.15 (Pin_15), U1.40 (GPIO35)
- new net IO36: J5.13 (Pin_13), U1.41 (GPIO36)
- new net IO37: J5.11 (Pin_11), U1.42 (GPIO37)
- new net IO38: J5.5 (Pin_5), U1.43 (GPIO38)
- new net IO39: J5.4 (Pin_4), U1.44 (MTCK)
- new net IO40: J5.6 (Pin_6), U1.45 (MTDO)
- new net IO41: J5.7 (Pin_7), U1.47 (MTDI)
- new net IO42: J5.12 (Pin_12), U1.48 (MTMS)
- new net IO45: J5.9 (Pin_9), R31.1, U1.51 (GPIO45)
- new net IO46: J5.8 (Pin_8), U1.52 (GPIO46)
- new net IO47: J5.14 (Pin_14), U1.37 (SPICLK_P)
- new net IO48: J5.18 (Pin_18), U1.36 (SPICLK_N)
- new net IO4/BAT: R12.2, R19.1, U1.9 (GPIO4)
- new net IO5: J3.6 (Pin_6), U1.10 (GPIO5)
- new net IO6: J3.1 (Pin_1), U1.11 (GPIO6)
- new net IO7: J3.7 (Pin_7), U1.12 (GPIO7)
- new net IO8: J3.8 (Pin_8), U1.13 (GPIO8)
- new net IO9: J3.2 (Pin_2), U1.14 (GPIO9)
- new net RX: J5.10 (Pin_10), U1.50 (U0RXD)
- new net SPICS0: U1.32 (SPICS0), U2.1 (~{CS})
- new net SPID: R26.2, U2.5 (DI/IO_{0})
- new net SPIHD: R30.2, U2.7 (~{HOLD}/~{RESET}/IO_{3})
- new net SPIQ: R27.2, U2.2 (DO/IO_{1})
- new net SPISCK: R28.2, U2.6 (CLK)
- new net SPIWP: R29.2, U2.3 (~{WP}/IO_{2})
- new net TX: J5.3 (Pin_3), R24.2
- new net USB_D+: J1.A6 (D+), J1.B6 (D+), R18.1, R18.2, U1.26 (GPIO20/USB_D+)
- new net USB_D-: J1.A7 (D-), J1.B7 (D-), R2.1, R2.2, U1.25 (GPIO19/USB_D-)
- new net VBAT: C2.1, C8.1, J2.2 (Pin_2), Q1.3 (D), R12.1, U3.3 (V_{BAT})
- new net VDD_SPI: C13.1, C32.1, U1.29 (VDD_SPI), U2.8 (VCC)
- new net VSYS: C7.1, D4.1 (K), Q1.2 (S), U4.3 (VI)
- new net XTAL32N: C37.1, U1.22 (XTAL_32K_N), Y1.1
- new net XTAL32P: C38.1, U1.21 (XTAL_32K_P), Y1.2
- no-connect marks 0 -> 1
Other:
- note added: "500mA"
- note added: "BATTERY CHARGER"
- note added: "HEADER PINS"
- note added: "IO45/IO46: pulldown~~{}"
- note added: "LEDS"
- note added: "MCU"
- note added: "MEMORY"
- note added: "POWER AND FILTERING"
- note added: "USB-C"
- note added: "VOLTAGE REGULATOR"
